Commit message: refine: so_arm urdf

File: config/so_100_arm.urdf.xacro (robot description, xacro)
@@ -4,5 +4,5 @@
     <xacro:arg name="use_fake_hardware" default="false"/>
     <!-- Import so_100_arm urdf file -->
-    <xacro:include filename="$(find so_100_arm)/urdf/so_100_arm.urdf" />
+    <xacro:include filename="$(find so_100_arm)/urdf/so_100_arm.xacro" />
     <!-- Import control_xacro -->
     <xacro:include filename="so_100_arm.ros2_control.xacro" />

File: urdf/so_100_arm.xacro (robot description, xacro)
@@ -1,14 +1,5 @@
-<?xml version="1.0" encoding="utf-8"?>
-<!-- This URDF was automatically created by SolidWorks to URDF Exporter! Originally created by Stephen Brawner (brawner@gmail.com)
-     Commit Version: 1.6.0-1-g15f4949  Build Version: 1.6.7594.29634
-     For more information, please see http://wiki.ros.org/sw_urdf_exporter -->
-<robot
-  name="so_100_arm">
-  <!-- <link name="world"/>
-  <joint name="world_to_base" type="fixed">
-    <parent link="world"/>
-    <child link="base_link"/>
-    <origin xyz="0 0 0" rpy="0 0 0"/>
-  </joint> -->
+<?xml version="1.0"?>
+<robot name="so_100_arm" xmlns:xacro="http://www.ros.org/wiki/xacro">
+  <xacro:property name="M_PI" value="3.1415926535897931" />
   <link
     name="base_link">
@@ -20,5 +11,5 @@
     <parent link="base_link"/>
     <child link="Base"/>
-    <origin xyz="0 0 0" rpy="0 0 0"/>
+    <origin xyz="0 0 0" rpy="0 0 ${M_PI/2}"/>
   </joint>
   <link
@@ -104,8 +95,8 @@
   <joint
     name="Shoulder_Rotation"
-    type="continuous">
+    type="revolute">
     <origin
       xyz="0 -0.0452 0.0165"
-      rpy="1.5708 0 0" />
+      rpy="${M_PI/2} 0 0" />
     <parent
       link="Base" />
@@ -114,4 +105,5 @@
     <axis
       xyz="0 1 0" />
+    <limit lower="${-M_PI/2}" upper="${M_PI/2}" effort="100" velocity="100"/>
   </joint>
   <link
@@ -157,5 +149,5 @@
   <joint
     name="Shoulder_Pitch"
-    type="continuous">
+    type="revolute">
     <origin
       xyz="0 0.1025 0.0306"
@@ -167,4 +159,5 @@
     <axis
       xyz="1 0 0" />
+    <limit lower="-1.8" upper="${M_PI/2}" effort="100" velocity="100"/>
   </joint>
   <link
@@ -210,5 +203,5 @@
   <joint
     name="Elbow"
-    type="continuous">
+    type="revolute">
     <origin
       xyz="0 0.11257 0.028"
@@ -220,4 +213,5 @@
     <axis
       xyz="1 0 0" />
+    <limit lower="${-M_PI/2}" upper="${M_PI/2}" effort="100" velocity="100"/>
   </joint>
   <link
@@ -263,5 +257,5 @@
   <joint
     name="Wrist_Pitch"
-    type="continuous">
+    type="revolute">
     <origin
       xyz="0 0.0052 0.1349"
@@ -273,4 +267,5 @@
     <axis
       xyz="1 0 0" />
+    <limit lower="${-M_PI}" upper="0" effort="100" velocity="100"/>
   </joint>
   <link
@@ -316,5 +311,5 @@
   <joint
     name="Wrist_Roll"
-    type="continuous">
+    type="revolute">
     <origin
       xyz="0 -0.0601 0"
@@ -326,4 +321,5 @@
     <axis
       xyz="0 1 0" />
+    <limit lower="${-M_PI}" upper="${M_PI}" effort="100" velocity="100"/>
   </joint>
   <link
@@ -369,5 +365,5 @@
   <joint
     name="Gripper"
-    type="continuous">
+    type="revolute">
     <origin
       xyz="-0.0202 -0.0244 0"
@@ -379,4 +375,11 @@
     <axis
       xyz="0 0 1" />
+    <limit lower="${-M_PI/20}" upper="${M_PI/2}" effort="100" velocity="100"/>
+  </joint>
+  <link name="tool0" />
+  <joint name="tool0_joint" type="fixed">
+    <parent link="Fixed_Gripper" />
+    <child link="tool0" />
+    <origin xyz="0 -0.1 0" rpy="0 0 ${-M_PI/2}" />
   </joint>
 </robot>
