Commit message: refine: initial_positions and gripper_controller

File: config/so_100_arm.ros2_control.xacro (robot description, xacro)
@@ -3,4 +3,6 @@
     <xacro:macro name="so_100_arm_ros2_control" params="name initial_positions_file use_fake_hardware" >
         <xacro:property name="initial_positions" value="${xacro.load_yaml(initial_positions_file)['initial_positions']}"/>
+        <xacro:property name="zero_positions" value="${xacro.load_yaml(initial_positions_file)['zero_positions']}"/>
+        <xacro:property name="directions" value="${xacro.load_yaml(initial_positions_file)['directions']}"/>
         <ros2_control name="${name}" type="system">
             <hardware>
@@ -20,5 +22,7 @@
                   <param name="initial_value">${initial_positions['Shoulder_Rotation']}</param>
                 </state_interface>
-                <!-- <state_interface name="velocity"/> -->
+                <state_interface name="velocity"/>
+                <param name="zero_position">${zero_positions['Shoulder_Rotation']}</param>
+                <param name="direction">${directions['Shoulder_Rotation']}</param>
             </joint>
             <joint name="Shoulder_Pitch">
@@ -27,5 +31,7 @@
                   <param name="initial_value">${initial_positions['Shoulder_Pitch']}</param>
                 </state_interface>
-                <!-- <state_interface name="velocity"/> -->
+                <state_interface name="velocity"/>
+                <param name="zero_position">${zero_positions['Shoulder_Pitch']}</param>
+                <param name="direction">${directions['Shoulder_Pitch']}</param>
             </joint>
             <joint name="Elbow">
@@ -34,5 +40,7 @@
                   <param name="initial_value">${initial_positions['Elbow']}</param>
                 </state_interface>
-                <!-- <state_interface name="velocity"/> -->
+                <state_interface name="velocity"/>
+                <param name="zero_position">${zero_positions['Elbow']}</param>
+                <param name="direction">${directions['Elbow']}</param>
             </joint>
             <joint name="Wrist_Pitch">
@@ -41,5 +49,7 @@
                   <param name="initial_value">${initial_positions['Wrist_Pitch']}</param>
                 </state_interface>
-                <!-- <state_interface name="velocity"/> -->
+                <state_interface name="velocity"/>
+                <param name="zero_position">${zero_positions['Wrist_Pitch']}</param>
+                <param name="direction">${directions['Wrist_Pitch']}</param>
             </joint>
             <joint name="Wrist_Roll">
@@ -48,5 +58,7 @@
                   <param name="initial_value">${initial_positions['Wrist_Roll']}</param>
                 </state_interface>
-                <!-- <state_interface name="velocity"/> -->
+                <state_interface name="velocity"/>
+                <param name="zero_position">${zero_positions['Wrist_Roll']}</param>
+                <param name="direction">${directions['Wrist_Roll']}</param>
             </joint>
             <joint name="Gripper">
@@ -55,5 +67,7 @@
                   <param name="initial_value">${initial_positions['Gripper']}</param>
                 </state_interface>
-                <!-- <state_interface name="velocity"/> -->
+                <state_interface name="velocity"/>
+                <param name="zero_position">${zero_positions['Gripper']}</param>
+                <param name="direction">${directions['Gripper']}</param>
             </joint>
         </ros2_control>

Commit message: refactor with motor_ids

File: config/so_100_arm.ros2_control.xacro (robot description, xacro)
@@ -3,4 +3,5 @@
     <xacro:macro name="so_100_arm_ros2_control" params="name initial_positions_file use_fake_hardware" >
         <xacro:property name="initial_positions" value="${xacro.load_yaml(initial_positions_file)['initial_positions']}"/>
+        <xacro:property name="motor_ids" value="${xacro.load_yaml(initial_positions_file)['motor_ids']}"/>
         <xacro:property name="zero_positions" value="${xacro.load_yaml(initial_positions_file)['zero_positions']}"/>
         <xacro:property name="directions" value="${xacro.load_yaml(initial_positions_file)['directions']}"/>
@@ -23,4 +24,5 @@
                 </state_interface>
                 <state_interface name="velocity"/>
+                <param name="motor_id">${motor_ids['Shoulder_Rotation']}</param>
                 <param name="zero_position">${zero_positions['Shoulder_Rotation']}</param>
                 <param name="direction">${directions['Shoulder_Rotation']}</param>
@@ -32,4 +34,5 @@
                 </state_interface>
                 <state_interface name="velocity"/>
+                <param name="motor_id">${motor_ids['Shoulder_Pitch']}</param>
                 <param name="zero_position">${zero_positions['Shoulder_Pitch']}</param>
                 <param name="direction">${directions['Shoulder_Pitch']}</param>
@@ -41,4 +44,5 @@
                 </state_interface>
                 <state_interface name="velocity"/>
+                <param name="motor_id">${motor_ids['Elbow']}</param>
                 <param name="zero_position">${zero_positions['Elbow']}</param>
                 <param name="direction">${directions['Elbow']}</param>
@@ -50,4 +54,5 @@
                 </state_interface>
                 <state_interface name="velocity"/>
+                <param name="motor_id">${motor_ids['Wrist_Pitch']}</param>
                 <param name="zero_position">${zero_positions['Wrist_Pitch']}</param>
                 <param name="direction">${directions['Wrist_Pitch']}</param>
@@ -59,4 +64,5 @@
                 </state_interface>
                 <state_interface name="velocity"/>
+                <param name="motor_id">${motor_ids['Wrist_Roll']}</param>
                 <param name="zero_position">${zero_positions['Wrist_Roll']}</param>
                 <param name="direction">${directions['Wrist_Roll']}</param>
@@ -68,4 +74,5 @@
                 </state_interface>
                 <state_interface name="velocity"/>
+                <param name="motor_id">${motor_ids['Gripper']}</param>
                 <param name="zero_position">${zero_positions['Gripper']}</param>
                 <param name="direction">${directions['Gripper']}</param>
